File: Hardware/Core.sch (KiCad schematic (older format))
At the start: 19 parts, among them U1 TM4C123GH6PZ

Commit message: Add bus pinout
Parts:
- removed C11, C2, C3, C4, C5, C6, C7, C8, C9: 0.1uF, CAPC1608, symbol C
- removed C? (x2): 20pF, CAPC1608, symbol C
- added C? (x12): 0.1uF, CAPC1005, symbol C
- added C? (x2): 20pF, CAPC1005, symbol C
- added J?: DEBUG-ARM-10, symbol DEBUG-ARM-10
- added R?: 1k, ~, symbol R
- added R?: R, ~, symbol R
- C?: renamed from C1; footprint CAPC1608 -> CAPC1005; Dielectric X5R -> D; Distributor Part No 399-5502-1-ND -> (none); MFR Name Kemet -> (none); MFR Part No C0603C335M9PACTU -> (none); Voltage >3V -> V
- C?: renamed from C10; footprint CAPC1608 -> CAPC1005; Dielectric X7R -> D; Distributor Part No 1276-1018-1-ND -> (none); MFR Name Samsung -> (none); MFR Part No CL10B102KB8NNNC -> (none); Voltage 50V -> V
- X?: value CRYSTAL -> 16MHz
- renumbered FB1 to FB?, U1 to U?
Connections:
- net labels added: +3.3VADC, +3.3VDAC, TCK, TDI, TDO, TMS, TRCLK, TRD0, TRD1, TRD2, TRD3, ~RST
- net labels removed: +3.3V, GNDA, REF+, REF-
- wire segments 68 -> 97
Other:
- moved on the sheet: C?, FB?, U?C, U?F, X?

Commit message: Save annotation
Parts:
- gave numbers to parts that had none: 25
