File: Hardware/CubeSat-Bus.sch (KiCad schematic (older format))
At the start: 1 part

Commit message: Rough pinout
Parts:
- renumbered H1 to H?
Connections:
- net +3.3VP: now also H?.1.27 (SENSE), H?.1.28 (VREF2); no longer H?.2.27 (3V3), H?.2.28 (3V3)
- net +5VP: now also H?.1.25 (~FAULT), H?.1.26 (VREF0); no longer H?.2.25 (5V), H?.2.26 (5V)
- net +BATT: now also H?.1.45, H?.1.46; no longer H?.2.45 (BATT), H?.2.46 (BATT)
- net ADCS0: now also H?.1.17 (IO.7); no longer H?.2.17 (IO.31)
- net ADCS1: now also H?.1.18 (IO.6); no longer H?.2.18 (IO.30)
- net ADCS2: now also H?.1.19 (IO.5); no longer H?.2.19 (IO.29)
- net ADCS3: now also H?.1.20 (IO.4); no longer H?.2.20 (IO.28)
- net ADCS4: now also H?.1.21 (IO.3); no longer H?.2.21 (IO.27)
- net ADCS5: now also H?.1.22 (IO.2); no longer H?.2.22 (IO.26)
- net ADCS6: now also H?.1.23 (IO.1); no longer H?.2.23 (IO.25)
- net ADCS7: now also H?.1.24 (IO.0); no longer H?.2.24 (IO.24)
- net AGND: now also H?.1.31 (OFF_V); no longer H?.2.31 (AGND)
- net COM0: now also H?.1.9 (IO.15); no longer H?.2.9 (IO.39)
- net COM1: now also H?.1.10 (IO.14); no longer H?.2.10 (IO.38)
- net COM2: now also H?.1.11 (IO.13); no longer H?.2.11 (IO.37)
- net COM3: now also H?.1.12 (IO.12); no longer H?.2.12 (IO.36)
- net COM4: now also H?.1.13 (IO.11); no longer H?.2.13 (IO.35)
- net COM5: now also H?.1.14 (IO.10); no longer H?.2.14 (IO.34)
- net COM6: now also H?.1.15 (IO.9); no longer H?.2.15 (IO.33)
- net COM7: now also H?.1.16 (IO.8); no longer H?.2.16 (IO.32)
- net DGND: now also H?.1.29 (~RESET), H?.1.30 (VREF1), H?.1.32 (VUSB); no longer H?.2.29 (DGND), H?.2.30 (DGND), H?.2.32 (DGND)
- net EPS0: now also H?.1.1 (IO.23); no longer H?.2.1 (IO.47)
- net EPS1: now also H?.1.2 (IO.22); no longer H?.2.2 (IO.46)
- net EPS2: now also H?.1.3 (IO.21); no longer H?.2.3 (IO.45)
- net EPS3: now also H?.1.4 (IO.20); no longer H?.2.4 (IO.44)
- net EPS4: now also H?.1.5 (IO.19); no longer H?.2.5 (IO.43)
- net EPS5: now also H?.1.6 (IO.18); no longer H?.2.6 (IO.42)
- net EPS6: now also H?.1.7 (IO.17); no longer H?.2.7 (IO.41)
- net EPS7: now also H?.1.8 (IO.16); no longer H?.2.8 (IO.40)
- net PAY0: now also H?.1.47 (USR0); no longer H?.2.47 (USR6)
- net PAY1: now also H?.1.48 (USR1); no longer H?.2.48 (USR7)
- net PAY2: now also H?.1.49 (USR2); no longer H?.2.49 (USR8)
- net PAY3: now also H?.1.50 (USR3); no longer H?.2.50 (USR9)
- net PAY4: now also H?.1.51 (USR4); no longer H?.2.51 (USR10)
- net PAY5: now also H?.1.52 (USR5); no longer H?.2.52 (USR11)
- net S0: now also H?.1.33 (VTCVR), H?.1.34 (RST); no longer H?.2.33 (S0), H?.2.34 (S0)
- net S1: now also H?.1.35 (CTS), H?.1.36 (RTS); no longer H?.2.35 (S1), H?.2.36 (S1)
- net S2: now also H?.1.37 (DSR), H?.1.38 (DTR); no longer H?.2.37 (S2), H?.2.38 (S2)
- net S3: now also H?.1.39 (TXD), H?.1.40 (RXD); no longer H?.2.39 (S3), H?.2.40 (S3)
- net S4: now also H?.1.41 (SDA), H?.1.42 (BCKUP); no longer H?.2.41 (S4), H?.2.42 (S4)
- net S5: now also H?.1.43 (SCL), H?.1.44; no longer H?.2.43 (S5), H?.2.44 (S5)
Changed lines of the file:
@@
 Sheet 2 4
 Title "Hyperion"
-Date "1 apr 2014"
+Date "29 apr 2014"
 Rev "0.2"
 Comp "Aerodyne Labs"
@@
 $EndDescr
 $Comp
-L CUBESAT-BUS H1
+L CUBESAT-BUS H?
 U 1 1 530D9DF3
 P 4200 4050
-F 0 "H1" H 4200 5400 60  0000 C CNN
+F 0 "H?" H 4200 5400 60  0000 C CNN
 F 1 "CUBESAT-BUS" H 4200 2700 60  0000 C CNN
 F 2 "~" H 4200 4050 60  0000 C CNN
@@
 $EndComp
 $Comp
-L CUBESAT-BUS H1
-U 2 1 530D9E02
+L CUBESAT-BUS H?
+U 1 1 530D9E02
 P 7200 4050
-F 0 "H1" H 7200 5400 60  0000 C CNN
+F 0 "H?" H 7200 5400 60  0000 C CNN
 F 1 "CUBESAT-BUS" H 7200 2700 60  0000 C CNN
 F 2 "~" H 7200 4050 60  0000 C CNN
 F 3 "~" H 7200 4050 60  0000 C CNN
-	2    7200 4050
+	1    7200 4050
 	1    0    0    -1
 $EndComp
@@
 	6100 4100 6600 4100
 $Comp
-L DGND #PWR01
+L DGND #PWR?
 U 1 1 530DA2E3
 P 8200 4200
-F 0 "#PWR01" H 8200 4200 40  0001 C CNN
+F 0 "#PWR?" H 8200 4200 40  0001 C CNN
 F 1 "DGND" H 8200 4130 40  0000 C CNN
 F 2 "" H 8200 4200 60  0000 C CNN
@@
 $EndComp
 $Comp
-L DGND #PWR02
+L DGND #PWR?
 U 1 1 530DA2F2
 P 6200 4200
-F 0 "#PWR02" H 6200 4200 40  0001 C CNN
+F 0 "#PWR?" H 6200 4200 40  0001 C CNN
 F 1 "DGND" H 6200 4130 40  0000 C CNN
 F 2 "" H 6200 4200 60  0000 C CNN
@@
 	6200 4200 6600 4200
 $Comp
-L AGND #PWR03
+L AGND #PWR?
 U 1 1 530DA31E
 P 6300 4300
-F 0 "#PWR03" H 6300 4300 40  0001 C CNN
+F 0 "#PWR?" H 6300 4300 40  0001 C CNN
 F 1 "AGND" H 6300 4230 50  0000 C CNN
 F 2 "" H 6300 4300 60  0000 C CNN
@@
 S5
 $Comp
-L +BATT #PWR04
+L +BATT #PWR?
 U 1 1 530DA395
 P 8300 5000
-F 0 "#PWR04" H 8300 4950 20  0001 C CNN
+F 0 "#PWR?" H 8300 4950 20  0001 C CNN
 F 1 "+BATT" H 8300 5100 30  0000 C CNN
 F 2 "" H 8300 5000 60  0000 C CNN
@@
 $EndComp
 $Comp
-L +BATT #PWR05
+L +BATT #PWR?
 U 1 1 530DA3A4
 P 6100 5000
-F 0 "#PWR05" H 6100 4950 20  0001 C CNN
+F 0 "#PWR?" H 6100 4950 20  0001 C CNN
 F 1 "+BATT" H 6100 5100 30  0000 C CNN
 F 2 "" H 6100 5000 60  0000 C CNN
@@
 	7800 5300 7900 5300
 $Comp
-L VMEM #PWR06
+L VMEM #PWR?
 U 1 1 530DA4D5
 P 5100 4800
-F 0 "#PWR06" H 5100 5000 40  0001 C CNN
+F 0 "#PWR?" H 5100 5000 40  0001 C CNN
 F 1 "VMEM" H 5100 4950 40  0000 C CNN
 F 2 "" H 5100 4800 60  0000 C CNN
@@
 NoConn ~ 3600 5000
 $Comp
-L VCOM #PWR1
+L VCOM #PWR?
 U 1 1 530DA51B
 P 5100 4300
-F 0 "#PWR1" H 5100 4500 40  0001 C CNN
+F 0 "#PWR?" H 5100 4500 40  0001 C CNN
 F 1 "VCOM" H 5100 4450 40  0000 C CNN
 F 2 "" H 5100 4300 60  0000 C CNN
@@
 	9000 1600 9100 1600
 $Comp
-L +5VP #PWR07
+L +5VP #PWR?
 U 1 1 530FA826
 P 6000 4000
-F 0 "#PWR07" H 6000 4090 20  0001 C CNN
+F 0 "#PWR?" H 6000 4090 20  0001 C CNN
 F 1 "+5VP" H 6000 4090 30  0000 C CNN
 F 2 "" H 6000 4000 60  0000 C CNN
@@
 $EndComp
 $Comp
-L +3.3VP #PWR08
+L +3.3VP #PWR?
 U 1 1 530FA83A
 P 6100 4100
-F 0 "#PWR08" H 6150 4130 20  0001 C CNN
+F 0 "#PWR?" H 6150 4130 20  0001 C CNN
 F 1 "+3.3VP" H 6100 4190 30  0000 C CNN
 F 2 "" H 6100 4100 60  0000 C CNN
@@
 $EndComp
 $Comp
-L +3.3VP #PWR09
+L +3.3VP #PWR?
 U 1 1 530FA867
 P 8300 4100
-F 0 "#PWR09" H 8350 4130 20  0001 C CNN
+F 0 "#PWR?" H 8350 4130 20  0001 C CNN
 F 1 "+3.3VP" H 8300 4190 30  0000 C CNN
 F 2 "" H 8300 4100 60  0000 C CNN
@@
 $EndComp
 $Comp
-L +5VP #PWR010
+L +5VP #PWR?
 U 1 1 530FA876
 P 8400 4000
-F 0 "#PWR010" H 8400 4090 20  0001 C CNN
+F 0 "#PWR?" H 8400 4090 20  0001 C CNN
 F 1 "+5VP" H 8400 4090 30  0000 C CNN
 F 2 "" H 8400 4000 60  0000 C CNN
