File: Hardware/Interface-Port.sch (KiCad schematic (older format))
At the start: 0 parts

Commit message: Rough USB interface
Parts:
- added C? (x2): C, CAPC1005-N, symbol C
- added C? (x11): 0.1uF, ~, symbol C
- added C?: 3.3uF, ~, symbol C
- added C? (x2): 4.7uF, ~, symbol C
- added D1, D2: TVS, CAPC1005-N, symbol TVS
- added FB? (x2): FERRITE, ~, symbol FERRITE
- added J1: CONN-DC, CONN-DC-CUI-202, symbol CONN-DC
- added J2: USB, CONN-USB-MICRO-B-FCI, symbol USB_MINI
- added R1, R2: MOV, RESC1005-N, symbol THERMISTOR
- added R?: 12k, ~, symbol R
- added R? (x4): 10k, RESC1005-N, symbol R
- added R?: 2.2k, ~, symbol R
- added R?: 4.7k, RESC1005-N, symbol R
- added R?: 10k, ~, symbol R
- added TH1: PTC, RESC1005-N, symbol THERMISTOR
- added U1: FT2232H, ~, symbol FT2232H
- added U?: 93LC46/OT, ~, symbol 93LC46/OT
- added X?: 12MHz, XTAL-4SMD-32X25, symbol CRYSTAL
Connections:
- net labels added: +1.8V, +3.3V, CLK, CS, D+, D-, DAT, GND, OSCI, OSCO, PwrSav, RST, RXD, RXLED, Reset, Shield, TCK, TDI, TDO, TMS, TXD, TXLED, VCOM
- wire segments 0 -> 126
- no-connect marks 0 -> 29

Commit message: Interface Component selection
Parts:
- removed C?: C, CAPC1005-N, symbol C
- removed C? (x10): 0.1uF, ~, symbol C
- removed C? (x2): 4.7uF, ~, symbol C
- removed R? (x3): 10k, RESC1005-N, symbol R
- removed R?: 4.7k, RESC1005-N, symbol R
- removed R?: 10k, ~, symbol R
- added C? (x10): 0.1uF, CAPC1005-N, symbol C
- added C? (x2): 3.3uF, CAPC1005-N, symbol C
- added C?: 27pF, CAPC1005-N, symbol C
- added R? (x5): 10k, RESC1005-N, symbol R
- C?: value C -> 27pF; Dielectric D -> NP0; Distributor Part No (none) -> 311-1019-1-ND; MFR Name (none) -> Yageo; MFR Part No (none) -> CC0402JRNPO9BN270; Voltage V -> 50V
- C?: footprint ~ -> CAPC1005-N; Dielectric D -> X5R; Distributor Part No (none) -> 1276-1443-1-ND; MFR Name (none) -> Samsung; MFR Part No (none) -> CL05A104MP5NNNC; Voltage V -> 10V
- C?: footprint ~ -> CAPC1005-N; Dielectric D -> X5R; Distributor Part No (none) -> 445-8022-1-ND; MFR Name (none) -> TDK; MFR Part No (none) -> C1005X5R1A335M050BC; Voltage V -> 10V
- R?: footprint ~ -> RESC1005-N; Distributor Part No (none) -> 311-12.0KLRCT-ND; MFR Name (none) -> Yageo; MFR Part No (none) -> RC0402FR-0712KL; Power W -> 1/16W
- R?: Distributor Part No (none) -> 311-10KJRCT-ND; MFR Name (none) -> Yageo; MFR Part No (none) -> RC0402JR-0710KL; Power W -> 1/16W; Tolerance % -> 5%
- R?: footprint ~ -> RESC1005-N; Distributor Part No (none) -> 311-2.2KJRCT-ND; MFR Name (none) -> Yageo; MFR Part No (none) -> 5%; Power W -> 1/16W; Tolerance % -> 5%
- TH?: renamed from TH1; footprint RESC1005-N -> RESC3216-N; Distributor Part No (none) -> 507-1802-1-ND; Hold Current (none) -> 0.5A; MFR Name (none) -> Bel Fuse; MFR Part No (none) -> 0ZCJ0050FF2G
- U1: Distributor Part No (none) -> 768-1024-1-ND; MFR Name (none) -> FTDI; MFR Part No (none) -> FT2232HL-REEL
- U2: renamed from U?; Distributor Part No (none) -> 93LC46BT-I/OTCT-ND; MFR Name (none) -> Microchip; MFR Part No (none) -> 93LC46BT-I/OT
- gave numbers to parts that had none: 1
- renumbered D1 to D?, D2 to D?, J2 to J1, J1 to J2, R1 to R?, R2 to R?
Connections:
- wire segments 126 -> 176
Other:
- moved on the sheet: C?, D?, FB?, X1

Commit message: Temporary annotation
Parts:
- removed FB?: FERRITE, ~, symbol FERRITE
- added FB1: 600, INDC1005-N, symbol FERRITE
- FB2: renamed from FB?; value FERRITE -> 600; footprint ~ -> INDC1005-N; Distributor Part No (none) -> 1276-6336-1-ND; MFR Name (none) -> Samsung; MFR Part No (none) -> CIM05U102NC
- U2: footprint ~ -> SOT95P280-6N
- gave numbers to parts that had none: 29
Connections:
- wire segments 176 -> 126

Commit message: Add protection circuit to DC jack
Parts:
- added Q1: MOSFET-P, SOT65P210-DDGSDD-N, symbol MOSFET-P
- added Q2: FDC6561, SOT95P280-6N, symbol MOSFET-N-DUAL
- added R11: 0.02, RESC3216-N, symbol R
- added U3: LTC4361-T, symbol LTC4361-T
Connections:
- wire segments 126 -> 148
Other:
- note added: "Rated -20C - 70C"
- note added: "Rated 0C - 70C"
Changed lines of the file:
@@
 Sheet 3 3
 Title ""
-Date "2 mar 2014"
+Date "4 mar 2014"
 Rev ""
 Comp ""
@@
 	1200 1700 2300 1700
 $Comp
-L VCOM #PWR25
+L VCOM #PWR27
 U 1 1 530FCA2A
 P 8700 2200
-F 0 "#PWR25" H 8700 2400 40  0001 C CNN
+F 0 "#PWR27" H 8700 2400 40  0001 C CNN
 F 1 "VCOM" H 8700 2350 40  0000 C CNN
 F 2 "" H 8700 2200 60  0000 C CNN
@@
 	0    -1   -1   0
 $EndComp
+$Comp
+L LTC4361-T U3
+U 1 1 53150BF6
+P 3700 7250
+F 0 "U3" H 3700 7500 60  0000 C CNN
+F 1 "LTC4361-T" H 3700 7000 60  0000 C CNN
+F 2 "" H 3750 7250 60  0000 C CNN
+F 3 "" H 3750 7250 60  0000 C CNN
+F 4 "Linear" H 3700 7250 60  0001 C CNN "MFR Name"
+F 5 "LTC4361CTS8-2#TRMPBF" H 3700 7250 60  0001 C CNN "MFR Part No"
+F 6 "LTC4361CTS8-2#TRMPBFCT-ND" H 3700 7250 60  0001 C CNN "Distributor Part No"
+	1    3700 7250
+	1    0    0    -1
+$EndComp
+$Comp
+L MOSFET-P Q1
+U 1 1 53150F21
+P 2100 6600
+F 0 "Q1" H 2000 6550 60  0000 R CNN
+F 1 "MOSFET-P" V 2300 6600 60  0000 C CNN
+F 2 "SOT65P210-DDGSDD-N" H 2100 6600 60  0001 C CNN
+F 3 "~" H 2100 6600 60  0000 C CNN
+F 4 "Vishay" H 2100 6600 60  0001 C CNN "MFR Name"
+F 5 "SI1471DH-T1-GE3" H 2100 6600 60  0001 C CNN "MFR Part No"
+F 6 "SI1471DH-T1-GE3CT-ND" H 2100 6600 60  0001 C CNN "Distributor Part No"
+	1    2100 6600
+	0    1    -1   0
+$EndComp
+$Comp
+L R R11
+U 1 1 53150F53
+P 2750 6500
+F 0 "R11" H 2750 6600 50  0000 C CNN
+F 1 "0.02" H 2750 6500 50  0000 C CNN
+F 2 "RESC3216-N" H 2750 6500 60  0001 C CNN
+F 3 "~" H 2750 6500 60  0000 C CNN
+F 4 "Ohmite" H 2750 6500 60  0001 C CNN "MFR Name"
+F 5 "MCS1632R020FER" H 2750 6500 60  0001 C CNN "MFR Part No"
+F 6 "MCS1632R020FERCT-ND" H 2750 6500 60  0001 C CNN "Distributor Part No"
+F 7 "1W" H 2750 6400 50  0001 C CNN "Power"
+F 8 "1%" H 2750 6300 50  0001 C CNN "Tolerance"
+	1    2750 6500
+	1    0    0    -1
+$EndComp
+Wire Wire Line
+	2300 6500 2500 6500
+Wire Wire Line
+	2400 6500 2400 7200
+Wire Wire Line
+	2400 7200 3200 7200
+Connection ~ 2400 6500
+$Comp
+L MOSFET-N-DUAL Q2
+U 2 1 53152246
+P 4000 6600
+F 0 "Q2" H 3900 6650 60  0000 R CNN
+F 1 "FDC6561" V 4200 6600 60  0000 C CNN
+F 2 "SOT95P280-6N" H 4000 6600 60  0001 C CNN
+F 3 "~" H 4000 6600 60  0000 C CNN
+F 4 "Fairchild" H 4000 6600 60  0001 C CNN "MFR Name"
+F 5 "FDC6561AN" H 4000 6600 60  0001 C CNN "MFR Part No"
+F 6 "FDC6561ANCT-ND" H 4000 6600 60  0001 C CNN "Distributor Part No"
+	2    4000 6600
+	0    1    -1   0
+$EndComp
+Wire Wire Line
+	3000 6500 3200 6500
+Wire Wire Line
+	3500 6800 3500 6900
+Wire Wire Line
+	3500 6900 4300 6900
+Wire Wire Line
+	3900 6900 3900 6800
+Wire Wire Line
+	3100 6500 3100 7100
+Wire Wire Line
+	3100 7100 3200 7100
+Connection ~ 3100 6500
+Wire Wire Line
+	3600 6500 3800 6500
+Wire Wire Line
+	4300 6900 4300 7100
+Wire Wire Line
+	4300 7100 4200 7100
+Connection ~ 3900 6900
+Wire Wire Line
+	4200 6500 4400 6500
+Wire Wire Line
+	4400 6500 4400 7200
+Wire Wire Line
+	4400 7200 4200 7200
+$Comp
+L GND #PWR035
+U 1 1 53152800
+P 4300 7500
+F 0 "#PWR035" H 4300 7500 30  0001 C CNN
+F 1 "GND" H 4300 7430 30  0001 C CNN
+F 2 "" H 4300 7500 60  0000 C CNN
+F 3 "" H 4300 7500 60  0000 C CNN
+	1    4300 7500
+	1    0    0    -1
+$EndComp
+Wire Wire Line
+	4200 7400 4300 7400
+Wire Wire Line
+	4300 7400 4300 7500
+Wire Wire Line
+	2200 6800 2200 7300
+Wire Wire Line
+	2200 7300 3200 7300
+$Comp
+L GND #PWR036
+U 1 1 5315298F
+P 3100 7500
+F 0 "#PWR036" H 3100 7500 30  0001 C CNN
+F 1 "GND" H 3100 7430 30  0001 C CNN
+F 2 "" H 3100 7500 60  0000 C CNN
+F 3 "" H 3100 7500 60  0000 C CNN
+	1    3100 7500
+	1    0    0    -1
+$EndComp
+Wire Wire Line
+	3100 7500 3100 7400
+Wire Wire Line
+	3100 7400 3200 7400
+Wire Wire Line
+	1700 6500 1900 6500
+$Comp
+L MOSFET-N-DUAL Q2
+U 1 1 53152FB6
+P 3400 6600
+F 0 "Q2" H 3300 6650 60  0000 R CNN
+F 1 "FDC6561" V 3600 6600 60  0000 C CNN
+F 2 "SOT95P280-6N" H 3400 6600 60  0001 C CNN
+F 3 "~" H 3400 6600 60  0000 C CNN
+F 4 "Fairchild" H 3400 6600 60  0001 C CNN "MFR Name"
+F 5 "FDC6561AN" H 3400 6600 60  0001 C CNN "MFR Part No"
+F 6 "FDC6561ANCT-ND" H 3400 6600 60  0001 C CNN "Distributor Part No"
+	1    3400 6600
+	0    -1   -1   0
+$EndComp
+Text Notes 3000 7500 2    60   ~ 0
+Rated 0C - 70C
+Text Notes 9700 3500 0    60   ~ 0
+Rated -20C - 70C
 $EndSCHEMATC

Commit message: Core support circuitry
Parts:
- C11, C14: value 27pF -> 10pF; Distributor Part No 311-1019-1-ND -> 311-1014-1-ND; MFR Part No CC0402JRNPO9BN270 -> CC0402JRNPO9BN100
- X1: Distributor Part No CTX839CT-ND -> 644-1173-1-ND; MFR Name CTS -> NDK; MFR Part No 403C35D12M00000 -> NX3225GA-12MHZ- STD-CRG-2
Other:
- note removed: "Rated -20C - 70C"
Changed lines of the file:
@@
 $Descr A4 11693 8268
 encoding utf-8
-Sheet 3 3
+Sheet 3 4
 Title ""
-Date "4 mar 2014"
+Date "12 mar 2014"
 Rev ""
 Comp ""
@@
 F 2 "XTAL-4SMD-32X25" H 10150 2600 60  0001 C CNN
 F 3 "~" H 10150 2600 60  0000 C CNN
-F 4 "CTS" H 10150 2600 60  0001 C CNN "MFR Name"
-F 5 "403C35D12M00000" H 10150 2600 60  0001 C CNN "MFR Part No"
-F 6 "CTX839CT-ND" H 10150 2600 60  0001 C CNN "Distributor Part No"
+F 4 "NDK" H 10150 2600 60  0001 C CNN "MFR Name"
+F 5 "NX3225GA-12MHZ- STD-CRG-2" H 10150 2600 60  0001 C CNN "MFR Part No"
+F 6 "644-1173-1-ND" H 10150 2600 60  0001 C CNN "Distributor Part No"
 	1    10150 2600
 	1    0    0    -1
@@
 P 9800 2950
 F 0 "C11" H 9850 3100 60  0000 L CNN
-F 1 "27pF" H 9850 2800 60  0000 L CNN
+F 1 "10pF" H 9850 2800 60  0000 L CNN
 F 2 "CAPC1005-N" H 9800 2950 60  0001 C CNN
 F 3 "~" H 9800 2950 60  0000 C CNN
 F 4 "Yageo" H 9800 2950 60  0001 C CNN "MFR Name"
-F 5 "CC0402JRNPO9BN270" H 9800 2950 60  0001 C CNN "MFR Part No"
-F 6 "311-1019-1-ND" H 9800 2950 60  0001 C CNN "Distributor Part No"
+F 5 "CC0402JRNPO9BN100" H 9800 2950 60  0001 C CNN "MFR Part No"
+F 6 "311-1014-1-ND" H 9800 2950 60  0001 C CNN "Distributor Part No"
 F 7 "50V" H 9750 2800 60  0001 R CNN "Voltage"
 F 8 "NP0" H 9750 3100 60  0001 R CNN "Dielectric"
@@
 $EndComp
 $Comp
-L C C14
-U 1 1 53132BAD
-P 10500 2950
-F 0 "C14" H 10550 3100 60  0000 L CNN
-F 1 "27pF" H 10550 2800 60  0000 L CNN
-F 2 "CAPC1005-N" H 10500 2950 60  0001 C CNN
-F 3 "~" H 10500 2950 60  0000 C CNN
-F 4 "Yageo" H 10500 2950 60  0001 C CNN "MFR Name"
-F 5 "CC0402JRNPO9BN270" H 10500 2950 60  0001 C CNN "MFR Part No"
-F 6 "311-1019-1-ND" H 10500 2950 60  0001 C CNN "Distributor Part No"
-F 7 "50V" H 10450 2800 60  0001 R CNN "Voltage"
-F 8 "NP0" H 10450 3100 60  0001 R CNN "Dielectric"
-	1    10500 2950
-	1    0    0    -1
-$EndComp
-$Comp
 L FERRITE FB1
 U 1 1 53133098
@@
 Text Notes 3000 7500 2    60   ~ 0
 Rated 0C - 70C
-Text Notes 9700 3500 0    60   ~ 0
-Rated -20C - 70C
+$Comp
+L C C14
+U 1 1 5320CBD8
+P 10500 2950
+F 0 "C14" H 10550 3100 60  0000 L CNN
+F 1 "10pF" H 10550 2800 60  0000 L CNN
+F 2 "CAPC1005-N" H 10500 2950 60  0001 C CNN
+F 3 "~" H 10500 2950 60  0000 C CNN
+F 4 "Yageo" H 10500 2950 60  0001 C CNN "MFR Name"
+F 5 "CC0402JRNPO9BN100" H 10500 2950 60  0001 C CNN "MFR Part No"
+F 6 "311-1014-1-ND" H 10500 2950 60  0001 C CNN "Distributor Part No"
+F 7 "50V" H 10450 2800 60  0001 R CNN "Voltage"
+F 8 "NP0" H 10450 3100 60  0001 R CNN "Dielectric"
+	1    10500 2950
+	1    0    0    -1
+$EndComp
 $EndSCHEMATC

Commit message: Switch to STM32F4 MCU
Connections:
- net labels added: TRST
Changed lines of the file:
@@
 Sheet 3 4
 Title ""
-Date "16 mar 2014"
+Date "17 mar 2014"
 Rev ""
 Comp ""
@@
 	1    0    0    -1
 $EndComp
+Text HLabel 5000 4500 0    60   Output ~ 0
+TRST
 $EndSCHEMATC
