File: Hardware/Interface-Port.sch (KiCad schematic (older format))
At the start: 40 parts, among them J1 USB, J2 CONN-DC, Q1 MOSFET-P, Q2 FDC6561, U1 FT2232H, U2 93LC46/OT, U3 LTC4361-T, X1 12MHz

Commit message: Clear core in prep for new MCU
Connections:
- net labels removed: TRST
- wire segments 148 -> 150
- no-connect marks 29 -> 28
Changed lines of the file:
@@
 encoding utf-8
 Sheet 3 4
-Title ""
-Date "17 mar 2014"
-Rev ""
-Comp ""
-Comment1 ""
+Title "Hyperion"
+Date "1 apr 2014"
+Rev "0.2"
+Comp "Aerodyne Labs"
+Comment1 "ethanharstad@gmail.com"
 Comment2 ""
 Comment3 ""
@@
 NoConn ~ 5100 4500
 NoConn ~ 5100 4600
-NoConn ~ 5100 4700
 NoConn ~ 5100 4800
 NoConn ~ 5100 4900
@@
 NoConn ~ 6400 5200
 NoConn ~ 6400 5300
-Text HLabel 5000 4600 0    60   Output ~ 0
+Text HLabel 3400 4400 0    60   Output ~ 0
 RST
 $Comp
@@
 	1    0    0    -1
 $EndComp
-Text HLabel 5000 4500 0    60   Output ~ 0
-TRST
+$Comp
+L GND #PWR?
+U 1 1 5329F06C
+P 5000 5700
+F 0 "#PWR?" H 5000 5700 30  0001 C CNN
+F 1 "GND" H 5000 5630 30  0001 C CNN
+F 2 "" H 5000 5700 60  0000 C CNN
+F 3 "" H 5000 5700 60  0000 C CNN
+	1    5000 5700
+	1    0    0    -1
+$EndComp
+Wire Wire Line
+	5000 5700 5000 4700
+Wire Wire Line
+	5000 4700 5100 4700
 $EndSCHEMATC

Commit message: Rough pinout
Parts:
- removed J2: CONN-DC, CONN-DC-CUI-202, symbol CONN-DC
- removed Q1: MOSFET-P, SOT65P210-DDGSDD-N, symbol MOSFET-P
- removed Q2: FDC6561, SOT95P280-6N, symbol MOSFET-N-DUAL
- removed R11: 0.02, RESC3216-N, symbol R
- removed U3: LTC4361-T, symbol LTC4361-T
- renumbered C11 to C?, C15 to C?, C6 to C?, C16 to C?, C13 to C?, C12 to C?, C10 to C?, C9 to C?, C8 to C?, C7 to C?, C5 to C?, C4 to C?, C2 to C?, C3 to C?, C1 to C?, C14 to C?, D1 to D?, D2 to D?, FB2 to FB?, FB1 to FB?, J1 to J?, R1 to R?, R2 to R?, R3 to R?, R10 to R?, R7 to R?, R8 to R?, R4 to R?, R9 to R?, R5 to R?, R6 to R?, TH1 to TH?, U1 to U?, U2 to U?, X1 to X?
Connections:
- wire segments 150 -> 128
Other:
- note removed: "Rated 0C - 70C"

Commit message: Add RBF switch prototype
Parts:
- added J?: RBF/CHRG, symbol CONN-DC-JACK
- added Q? (x2): MOSFET-P, ~, symbol MOSFET-P
- added Q?: MOSFET-N, ~, symbol MOSFET-N
- added R? (x2): 10k, RESC1005-N, symbol R
- added TH?: THERMISTOR, ~, symbol THERMISTOR
- D? (x2): value TVS -> 40V
- R? (x2): value MOV -> 5.5V
- TH?: value PTC -> 0.5A
Connections:
- net labels added: DEP-C, DEP-NC, DEP-NO, RBF-C, RBF-NC, RBF-NO, S0, S1, S2, S3, S4, S5, VExt, VUsb
- wire segments 128 -> 155
Other:
- note added: "MOV"
- note added: "TVS"
- note added: "USB Transient Protection"
